Commit message: add sonar topics

File: robot_description/urdf/metal.xacro (robot description, xacro)
@@ -46,7 +46,7 @@
     <child link="xv11"/>
 <!--    plastic model     -->
-<origin xyz="-0.022 0 ${radius_wheel+0.135}" rpy="0 0 0"/>
+<!--<origin xyz="-0.022 0 ${radius_wheel+0.135}" rpy="0 0 0"/>-->
 <!--	metal model	-->
-<!--	<origin xyz="0.07 0 ${radius_wheel+0.135}" rpy="0 0 0"/>-->
+<origin xyz="0.07 0 ${radius_wheel+0.135}" rpy="0 0 0"/>
   </joint>
 <joint name="IMU_joint" type="fixed">
@@ -1019,5 +1019,5 @@
     </sensor>
   </gazebo>
- <!-- Proximity sensor plugin TO DO-->
+<!-- Proximity sensor plugin TO DO-->
   <gazebo reference="sonar_1">
     <sensor name ="sonar1" type="ray">
@@ -1082,5 +1082,5 @@
         <range>
           <min>0.02</min>
-          <max>3</max>
+          <max>4</max>
           <resolution>1</resolution>
         </range>
