Commit message: add lib map

File: robot_description/urdf/andbot_plastic.xacro (robot description, xacro)
@@ -21,5 +21,5 @@
       <origin xyz="0 0 -0.019" rpy="1.57 0 -1.57"/>
       <geometry>
-        <mesh filename="package://hyperlync_robot/robot_description/mesh/lidar_XV-11.STL"/>
+        <mesh filename="package://andbot_gazebo/robot_description/mesh/lidar_XV-11.STL"/>
       </geometry>
     </collision>
@@ -27,5 +27,5 @@
       <origin xyz="0 0 -0.019" rpy="1.57 0 -1.57"/>
       <geometry>
-        <mesh filename="package://hyperlync_robot/robot_description/mesh/lidar_XV-11.STL"/>
+        <mesh filename="package://andbot_gazebo/robot_description/mesh/lidar_XV-11.STL"/>
       </geometry>
        <material name="Green">
@@ -81,5 +81,5 @@
       <origin xyz="0 0 ${radius_wheel-height_wheels_from_base}" rpy="0 0 0"/>
       <geometry>
-        <mesh filename="package://hyperlync_robot/robot_description/mesh/base_part.STL"/>
+        <mesh filename="package://andbot_gazebo/robot_description/mesh/base_part.STL"/>
       </geometry>
     </collision>
@@ -87,5 +87,5 @@
       <origin xyz="0 0 ${radius_wheel-height_wheels_from_base}" rpy="0 0 0"/>
       <geometry>
-        <mesh filename="package://hyperlync_robot/robot_description/mesh/base_part.STL"/>
+        <mesh filename="package://andbot_gazebo/robot_description/mesh/base_part.STL"/>
       </geometry>
        <material name="Orange">
@@ -147,11 +147,11 @@
       <origin xyz="0 0 0" rpy="0 0 0"/>
       <geometry>
-        <mesh filename="package://hyperlync_robot/robot_description/mesh/fake_body.STL"/>
-      </geometry>
-    </collision>
-    <visual>
-      <origin xyz="0 0 0" rpy="0 0 0"/>
-      <geometry>
-        <mesh filename="package://hyperlync_robot/robot_description/mesh/fake_body.STL"/>
+        <mesh filename="package://andbot_gazebo/robot_description/mesh/fake_body.STL"/>
+      </geometry>
+    </collision>
+    <visual>
+      <origin xyz="0 0 0" rpy="0 0 0"/>
+      <geometry>
+        <mesh filename="package://andbot_gazebo/robot_description/mesh/fake_body.STL"/>
       </geometry>
        <material name="Blue">
@@ -178,11 +178,11 @@
       <origin xyz="0 0 0" rpy="0 0 0"/>
       <geometry>
-        <mesh filename="package://hyperlync_robot/robot_description/mesh/head.STL"/>
-      </geometry>
-    </collision>
-    <visual>
-      <origin xyz="0 0 0" rpy="0 0 0"/>
-      <geometry>
-        <mesh filename="package://hyperlync_robot/robot_description/mesh/head.STL"/>
+        <mesh filename="package://andbot_gazebo/robot_description/mesh/head.STL"/>
+      </geometry>
+    </collision>
+    <visual>
+      <origin xyz="0 0 0" rpy="0 0 0"/>
+      <geometry>
+        <mesh filename="package://andbot_gazebo/robot_description/mesh/head.STL"/>
       </geometry>
        <material name="Blue">
@@ -224,5 +224,5 @@
       <origin xyz="0 0 0" rpy="-1.5707 1.5707 0"/>
       <geometry>
-        <mesh filename="package://hyperlync_robot/robot_description/mesh/arm_link1.STL"/>
+        <mesh filename="package://andbot_gazebo/robot_description/mesh/arm_link1.STL"/>
       </geometry>
     </collision>
@@ -230,5 +230,5 @@
       <origin xyz="0 0 0" rpy="-1.5707 1.5707 0"/>
       <geometry>
-        <mesh filename="package://hyperlync_robot/robot_description/mesh/arm_link1.STL"/>
+        <mesh filename="package://andbot_gazebo/robot_description/mesh/arm_link1.STL"/>
       </geometry>
        <material name="Blue">
@@ -256,5 +256,5 @@
       <origin xyz="0 0 0" rpy="-1.5707 1.5707 0"/>
       <geometry>
-        <mesh filename="package://hyperlync_robot/robot_description/mesh/arm_link2.STL"/>
+        <mesh filename="package://andbot_gazebo/robot_description/mesh/arm_link2.STL"/>
       </geometry>
     </collision>
@@ -262,5 +262,5 @@
       <origin xyz="0 0 0" rpy="-1.5707 1.5707 0"/>
       <geometry>
-        <mesh filename="package://hyperlync_robot/robot_description/mesh/arm_link2.STL"/>
+        <mesh filename="package://andbot_gazebo/robot_description/mesh/arm_link2.STL"/>
       </geometry>
        <material name="Blue">
@@ -288,5 +288,5 @@
       <origin xyz="0 0 0" rpy="1.57 1.5707 0"/>
       <geometry>
-        <mesh filename="package://hyperlync_robot/robot_description/mesh/arm_link1.STL"/>
+        <mesh filename="package://andbot_gazebo/robot_description/mesh/arm_link1.STL"/>
       </geometry>
     </collision>
@@ -294,5 +294,5 @@
       <origin xyz="0 0 0" rpy="1.57 1.5707 0"/>
       <geometry>
-        <mesh filename="package://hyperlync_robot/robot_description/mesh/arm_link1.STL"/>
+        <mesh filename="package://andbot_gazebo/robot_description/mesh/arm_link1.STL"/>
       </geometry>
        <material name="Blue">
@@ -320,5 +320,5 @@
       <origin xyz="0 0 0" rpy="-1.5707 1.5707 3.14"/>
       <geometry>
-        <mesh filename="package://hyperlync_robot/robot_description/mesh/arm_link2.STL"/>
+        <mesh filename="package://andbot_gazebo/robot_description/mesh/arm_link2.STL"/>
       </geometry>
     </collision>
@@ -326,5 +326,5 @@
       <origin xyz="0 0 0" rpy="-1.5707 1.5707 0"/>
       <geometry>
-        <mesh filename="package://hyperlync_robot/robot_description/mesh/arm_link2.STL"/>
+        <mesh filename="package://andbot_gazebo/robot_description/mesh/arm_link2.STL"/>
       </geometry>
        <material name="Blue">
@@ -384,5 +384,5 @@
       <origin xyz="0 0 0" rpy="0 1.570795 1.570795"/>
       <geometry>
-        <mesh filename="package://hyperlync_robot/robot_description/mesh/wheel-D152_SMALL.STL"/>
+        <mesh filename="package://andbot_gazebo/robot_description/mesh/wheel-D152_SMALL.STL"/>
       </geometry>
     </collision>
@@ -390,5 +390,5 @@
       <origin xyz="0 0 0" rpy="0 1.570795 1.570795"/>
       <geometry>
-        <mesh filename="package://hyperlync_robot/robot_description/mesh/wheel-D152_SMALL.STL"/>
+        <mesh filename="package://andbot_gazebo/robot_description/mesh/wheel-D152_SMALL.STL"/>
       </geometry>
        <material name="Black">
@@ -435,5 +435,5 @@
       <origin xyz="0 0 0" rpy="0 1.570795 1.570795"/>
       <geometry>
-        <mesh filename="package://hyperlync_robot/robot_description/mesh/wheel-D152_SMALL.STL"/>
+        <mesh filename="package://andbot_gazebo/robot_description/mesh/wheel-D152_SMALL.STL"/>
       </geometry>
     </collision>
@@ -441,5 +441,5 @@
       <origin xyz="0 0 0" rpy="0 1.570795 1.570795"/>
       <geometry>
-        <mesh filename="package://hyperlync_robot/robot_description/mesh/wheel-D152_SMALL.STL"/>
+        <mesh filename="package://andbot_gazebo/robot_description/mesh/wheel-D152_SMALL.STL"/>
       </geometry>
        <material name="Black">
@@ -493,11 +493,11 @@
       <origin xyz="0 0 0" rpy="0 0 0"/>
       <geometry>
-        <mesh filename="package://hyperlync_robot/robot_description/mesh/sonar_HC_SR04.STL"/>
-      </geometry>
-    </collision>
-    <visual>
-      <origin xyz="0 0 0" rpy="0 0 0"/>
-      <geometry>
-        <mesh filename="package://hyperlync_robot/robot_description/mesh/sonar_HC_SR04.STL"/>
+        <mesh filename="package://andbot_gazebo/robot_description/mesh/sonar_HC_SR04.STL"/>
+      </geometry>
+    </collision>
+    <visual>
+      <origin xyz="0 0 0" rpy="0 0 0"/>
+      <geometry>
+        <mesh filename="package://andbot_gazebo/robot_description/mesh/sonar_HC_SR04.STL"/>
       </geometry>
        <material name="Yellow">
@@ -530,11 +530,11 @@
       <origin xyz="0 0 0" rpy="0 0 0"/>
       <geometry>
-        <mesh filename="package://hyperlync_robot/robot_description/mesh/sonar_HC_SR04.STL"/>
-      </geometry>
-    </collision>
-    <visual>
-      <origin xyz="0 0 0" rpy="0 0 0"/>
-      <geometry>
-        <mesh filename="package://hyperlync_robot/robot_description/mesh/sonar_HC_SR04.STL"/>
+        <mesh filename="package://andbot_gazebo/robot_description/mesh/sonar_HC_SR04.STL"/>
+      </geometry>
+    </collision>
+    <visual>
+      <origin xyz="0 0 0" rpy="0 0 0"/>
+      <geometry>
+        <mesh filename="package://andbot_gazebo/robot_description/mesh/sonar_HC_SR04.STL"/>
       </geometry>
        <material name="Yellow">
@@ -566,11 +566,11 @@
       <origin xyz="0 0 0" rpy="0 0 0"/>
       <geometry>
-        <mesh filename="package://hyperlync_robot/robot_description/mesh/sonar_HC_SR04.STL"/>
-      </geometry>
-    </collision>
-    <visual>
-      <origin xyz="0 0 0" rpy="0 0 0"/>
-      <geometry>
-        <mesh filename="package://hyperlync_robot/robot_description/mesh/sonar_HC_SR04.STL"/>
+        <mesh filename="package://andbot_gazebo/robot_description/mesh/sonar_HC_SR04.STL"/>
+      </geometry>
+    </collision>
+    <visual>
+      <origin xyz="0 0 0" rpy="0 0 0"/>
+      <geometry>
+        <mesh filename="package://andbot_gazebo/robot_description/mesh/sonar_HC_SR04.STL"/>
       </geometry>
        <material name="Yellow">
@@ -602,11 +602,11 @@
       <origin xyz="0 0 0" rpy="0 0 0"/>
       <geometry>
-        <mesh filename="package://hyperlync_robot/robot_description/mesh/sonar_HC_SR04.STL"/>
-      </geometry>
-    </collision>
-    <visual>
-      <origin xyz="0 0 0" rpy="0 0 0"/>
-      <geometry>
-        <mesh filename="package://hyperlync_robot/robot_description/mesh/sonar_HC_SR04.STL"/>
+        <mesh filename="package://andbot_gazebo/robot_description/mesh/sonar_HC_SR04.STL"/>
+      </geometry>
+    </collision>
+    <visual>
+      <origin xyz="0 0 0" rpy="0 0 0"/>
+      <geometry>
+        <mesh filename="package://andbot_gazebo/robot_description/mesh/sonar_HC_SR04.STL"/>
       </geometry>
        <material name="Yellow">
@@ -638,11 +638,11 @@
       <origin xyz="0 0 0" rpy="0 0 0"/>
       <geometry>
-        <mesh filename="package://hyperlync_robot/robot_description/mesh/sonar_HC_SR04.STL"/>
-      </geometry>
-    </collision>
-    <visual>
-      <origin xyz="0 0 0" rpy="0 0 0"/>
-      <geometry>
-        <mesh filename="package://hyperlync_robot/robot_description/mesh/sonar_HC_SR04.STL"/>
+        <mesh filename="package://andbot_gazebo/robot_description/mesh/sonar_HC_SR04.STL"/>
+      </geometry>
+    </collision>
+    <visual>
+      <origin xyz="0 0 0" rpy="0 0 0"/>
+      <geometry>
+        <mesh filename="package://andbot_gazebo/robot_description/mesh/sonar_HC_SR04.STL"/>
       </geometry>
        <material name="Yellow">
@@ -674,11 +674,11 @@
       <origin xyz="0 0 0" rpy="0 0 0"/>
       <geometry>
-        <mesh filename="package://hyperlync_robot/robot_description/mesh/sonar_HC_SR04.STL"/>
-      </geometry>
-    </collision>
-    <visual>
-      <origin xyz="0 0 0" rpy="0 0 0"/>
-      <geometry>
-        <mesh filename="package://hyperlync_robot/robot_description/mesh/sonar_HC_SR04.STL"/>
+        <mesh filename="package://andbot_gazebo/robot_description/mesh/sonar_HC_SR04.STL"/>
+      </geometry>
+    </collision>
+    <visual>
+      <origin xyz="0 0 0" rpy="0 0 0"/>
+      <geometry>
+        <mesh filename="package://andbot_gazebo/robot_description/mesh/sonar_HC_SR04.STL"/>
       </geometry>
        <material name="Yellow">
@@ -710,11 +710,11 @@
       <origin xyz="0 0 0" rpy="0 0 0"/>
       <geometry>
-        <mesh filename="package://hyperlync_robot/robot_description/mesh/sonar_HC_SR04.STL"/>
-      </geometry>
-    </collision>
-    <visual>
-      <origin xyz="0 0 0" rpy="0 0 0"/>
-      <geometry>
-        <mesh filename="package://hyperlync_robot/robot_description/mesh/sonar_HC_SR04.STL"/>
+        <mesh filename="package://andbot_gazebo/robot_description/mesh/sonar_HC_SR04.STL"/>
+      </geometry>
+    </collision>
+    <visual>
+      <origin xyz="0 0 0" rpy="0 0 0"/>
+      <geometry>
+        <mesh filename="package://andbot_gazebo/robot_description/mesh/sonar_HC_SR04.STL"/>
       </geometry>
        <material name="Yellow">
@@ -746,11 +746,11 @@
       <origin xyz="0 0 0" rpy="0 0 0"/>
       <geometry>
-        <mesh filename="package://hyperlync_robot/robot_description/mesh/sonar_HC_SR04.STL"/>
-      </geometry>
-    </collision>
-    <visual>
-      <origin xyz="0 0 0" rpy="0 0 0"/>
-      <geometry>
-        <mesh filename="package://hyperlync_robot/robot_description/mesh/sonar_HC_SR04.STL"/>
+        <mesh filename="package://andbot_gazebo/robot_description/mesh/sonar_HC_SR04.STL"/>
+      </geometry>
+    </collision>
+    <visual>
+      <origin xyz="0 0 0" rpy="0 0 0"/>
+      <geometry>
+        <mesh filename="package://andbot_gazebo/robot_description/mesh/sonar_HC_SR04.STL"/>
       </geometry>
        <material name="Yellow">
@@ -782,11 +782,11 @@
       <origin xyz="0 0 0" rpy="0 0 0"/>
       <geometry>
-        <mesh filename="package://hyperlync_robot/robot_description/mesh/sonar_HC_SR04.STL"/>
-      </geometry>
-    </collision>
-    <visual>
-      <origin xyz="0 0 0" rpy="0 0 0"/>
-      <geometry>
-        <mesh filename="package://hyperlync_robot/robot_description/mesh/sonar_HC_SR04.STL"/>
+        <mesh filename="package://andbot_gazebo/robot_description/mesh/sonar_HC_SR04.STL"/>
+      </geometry>
+    </collision>
+    <visual>
+      <origin xyz="0 0 0" rpy="0 0 0"/>
+      <geometry>
+        <mesh filename="package://andbot_gazebo/robot_description/mesh/sonar_HC_SR04.STL"/>
       </geometry>
        <material name="Yellow">
@@ -818,11 +818,11 @@
       <origin xyz="0 0 0" rpy="0 0 0"/>
       <geometry>
-        <mesh filename="package://hyperlync_robot/robot_description/mesh/sonar_HC_SR04.STL"/>
-      </geometry>
-    </collision>
-    <visual>
-      <origin xyz="0 0 0" rpy="0 0 0"/>
-      <geometry>
-        <mesh filename="package://hyperlync_robot/robot_description/mesh/sonar_HC_SR04.STL"/>
+        <mesh filename="package://andbot_gazebo/robot_description/mesh/sonar_HC_SR04.STL"/>
+      </geometry>
+    </collision>
+    <visual>
+      <origin xyz="0 0 0" rpy="0 0 0"/>
+      <geometry>
+        <mesh filename="package://andbot_gazebo/robot_description/mesh/sonar_HC_SR04.STL"/>
       </geometry>
        <material name="Yellow">
@@ -854,11 +854,11 @@
       <origin xyz="0 0 0" rpy="0 0 0"/>
       <geometry>
-        <mesh filename="package://hyperlync_robot/robot_description/mesh/sonar_HC_SR04.STL"/>
-      </geometry>
-    </collision>
-    <visual>
-      <origin xyz="0 0 0" rpy="0 0 0"/>
-      <geometry>
-        <mesh filename="package://hyperlync_robot/robot_description/mesh/sonar_HC_SR04.STL"/>
+        <mesh filename="package://andbot_gazebo/robot_description/mesh/sonar_HC_SR04.STL"/>
+      </geometry>
+    </collision>
+    <visual>
+      <origin xyz="0 0 0" rpy="0 0 0"/>
+      <geometry>
+        <mesh filename="package://andbot_gazebo/robot_description/mesh/sonar_HC_SR04.STL"/>
       </geometry>
        <material name="Yellow">
@@ -890,11 +890,11 @@
       <origin xyz="0 0 0" rpy="0 0 0"/>
       <geometry>
-        <mesh filename="package://hyperlync_robot/robot_description/mesh/sonar_HC_SR04.STL"/>
-      </geometry>
-    </collision>
-    <visual>
-      <origin xyz="0 0 0" rpy="0 0 0"/>
-      <geometry>
-        <mesh filename="package://hyperlync_robot/robot_description/mesh/sonar_HC_SR04.STL"/>
+        <mesh filename="package://andbot_gazebo/robot_description/mesh/sonar_HC_SR04.STL"/>
+      </geometry>
+    </collision>
+    <visual>
+      <origin xyz="0 0 0" rpy="0 0 0"/>
+      <geometry>
+        <mesh filename="package://andbot_gazebo/robot_description/mesh/sonar_HC_SR04.STL"/>
       </geometry>
        <material name="Yellow">
