Commit message: add lib map

File: robot_description/urdf/metal.xacro (robot description, xacro)
@@ -21,5 +21,5 @@
       <origin xyz="0 0 -0.019" rpy="1.57 0 -1.57"/>
       <geometry>
-        <mesh filename="package://andbot_gazebo/robot_description/mesh/lidar_XV-11.STL"/>
+        <mesh filename="package://hyperlync_robot/robot_description/mesh/lidar_XV-11.STL"/>
       </geometry>
     </collision>
@@ -27,5 +27,5 @@
       <origin xyz="0 0 -0.019" rpy="1.57 0 -1.57"/>
       <geometry>
-        <mesh filename="package://andbot_gazebo/robot_description/mesh/lidar_XV-11.STL"/>
+        <mesh filename="package://hyperlync_robot/robot_description/mesh/lidar_XV-11.STL"/>
       </geometry>
        <material name="Green">
@@ -46,7 +46,7 @@
     <child link="xv11"/>
 <!--    plastic model     -->
-<origin xyz="-0.022 0 ${radius_wheel+0.135}" rpy="0 0 0"/>
+<!--<origin xyz="-0.022 0 ${radius_wheel+0.135}" rpy="0 0 0"/>-->
 <!--	metal model	-->
-<!--	<origin xyz="0.07 0 ${radius_wheel+0.135}" rpy="0 0 0"/>-->
+<origin xyz="0.07 0 ${radius_wheel+0.135}" rpy="0 0 0"/>
   </joint>
 <joint name="IMU_joint" type="fixed">
@@ -81,5 +81,5 @@
       <origin xyz="0 0 ${radius_wheel-height_wheels_from_base}" rpy="0 0 0"/>
       <geometry>
-        <mesh filename="package://andbot_gazebo/robot_description/mesh/base_part.STL"/>
+        <mesh filename="package://hyperlync_robot/robot_description/mesh/base_part.STL"/>
       </geometry>
     </collision>
@@ -87,5 +87,5 @@
       <origin xyz="0 0 ${radius_wheel-height_wheels_from_base}" rpy="0 0 0"/>
       <geometry>
-        <mesh filename="package://andbot_gazebo/robot_description/mesh/base_part.STL"/>
+        <mesh filename="package://hyperlync_robot/robot_description/mesh/base_part.STL"/>
       </geometry>
        <material name="Orange">
@@ -95,5 +95,5 @@
     <inertial>
       <origin xyz="0 0 0.07" rpy="0 0 0"/>
-      <mass value="25"/>
+      <mass value="52"/>
       <inertia ixx="0.248" ixy="0" ixz="0" iyy="0.748" iyz="0" izz="0.748"/>
     </inertial>
@@ -131,6 +131,6 @@
   </link>
   <gazebo reference="caster_wheel">
-   <!-- <mu1>0.04</mu1>
-    <mu2>0.04</mu2>-->
+    <mu1>0.04</mu1>
+    <mu2>0.04</mu2>
     <material>Gazebo/White</material>
   </gazebo>
@@ -147,11 +147,11 @@
       <origin xyz="0 0 0" rpy="0 0 0"/>
       <geometry>
-        <mesh filename="package://andbot_gazebo/robot_description/mesh/fake_body.STL"/>
-      </geometry>
-    </collision>
-    <visual>
-      <origin xyz="0 0 0" rpy="0 0 0"/>
-      <geometry>
-        <mesh filename="package://andbot_gazebo/robot_description/mesh/fake_body.STL"/>
+        <mesh filename="package://hyperlync_robot/robot_description/mesh/fake_body.STL"/>
+      </geometry>
+    </collision>
+    <visual>
+      <origin xyz="0 0 0" rpy="0 0 0"/>
+      <geometry>
+        <mesh filename="package://hyperlync_robot/robot_description/mesh/fake_body.STL"/>
       </geometry>
        <material name="Blue">
@@ -178,11 +178,11 @@
       <origin xyz="0 0 0" rpy="0 0 0"/>
       <geometry>
-        <mesh filename="package://andbot_gazebo/robot_description/mesh/head.STL"/>
-      </geometry>
-    </collision>
-    <visual>
-      <origin xyz="0 0 0" rpy="0 0 0"/>
-      <geometry>
-        <mesh filename="package://andbot_gazebo/robot_description/mesh/head.STL"/>
+        <mesh filename="package://hyperlync_robot/robot_description/mesh/head.STL"/>
+      </geometry>
+    </collision>
+    <visual>
+      <origin xyz="0 0 0" rpy="0 0 0"/>
+      <geometry>
+        <mesh filename="package://hyperlync_robot/robot_description/mesh/head.STL"/>
       </geometry>
        <material name="Blue">
@@ -224,5 +224,5 @@
       <origin xyz="0 0 0" rpy="-1.5707 1.5707 0"/>
       <geometry>
-        <mesh filename="package://andbot_gazebo/robot_description/mesh/arm_link1.STL"/>
+        <mesh filename="package://hyperlync_robot/robot_description/mesh/arm_link1.STL"/>
       </geometry>
     </collision>
@@ -230,5 +230,5 @@
       <origin xyz="0 0 0" rpy="-1.5707 1.5707 0"/>
       <geometry>
-        <mesh filename="package://andbot_gazebo/robot_description/mesh/arm_link1.STL"/>
+        <mesh filename="package://hyperlync_robot/robot_description/mesh/arm_link1.STL"/>
       </geometry>
        <material name="Blue">
@@ -256,5 +256,5 @@
       <origin xyz="0 0 0" rpy="-1.5707 1.5707 0"/>
       <geometry>
-        <mesh filename="package://andbot_gazebo/robot_description/mesh/arm_link2.STL"/>
+        <mesh filename="package://hyperlync_robot/robot_description/mesh/arm_link2.STL"/>
       </geometry>
     </collision>
@@ -262,5 +262,5 @@
       <origin xyz="0 0 0" rpy="-1.5707 1.5707 0"/>
       <geometry>
-        <mesh filename="package://andbot_gazebo/robot_description/mesh/arm_link2.STL"/>
+        <mesh filename="package://hyperlync_robot/robot_description/mesh/arm_link2.STL"/>
       </geometry>
        <material name="Blue">
@@ -288,5 +288,5 @@
       <origin xyz="0 0 0" rpy="1.57 1.5707 0"/>
       <geometry>
-        <mesh filename="package://andbot_gazebo/robot_description/mesh/arm_link1.STL"/>
+        <mesh filename="package://hyperlync_robot/robot_description/mesh/arm_link1.STL"/>
       </geometry>
     </collision>
@@ -294,5 +294,5 @@
       <origin xyz="0 0 0" rpy="1.57 1.5707 0"/>
       <geometry>
-        <mesh filename="package://andbot_gazebo/robot_description/mesh/arm_link1.STL"/>
+        <mesh filename="package://hyperlync_robot/robot_description/mesh/arm_link1.STL"/>
       </geometry>
        <material name="Blue">
@@ -320,5 +320,5 @@
       <origin xyz="0 0 0" rpy="-1.5707 1.5707 3.14"/>
       <geometry>
-        <mesh filename="package://andbot_gazebo/robot_description/mesh/arm_link2.STL"/>
+        <mesh filename="package://hyperlync_robot/robot_description/mesh/arm_link2.STL"/>
       </geometry>
     </collision>
@@ -326,5 +326,5 @@
       <origin xyz="0 0 0" rpy="-1.5707 1.5707 0"/>
       <geometry>
-        <mesh filename="package://andbot_gazebo/robot_description/mesh/arm_link2.STL"/>
+        <mesh filename="package://hyperlync_robot/robot_description/mesh/arm_link2.STL"/>
       </geometry>
        <material name="Blue">
@@ -384,5 +384,5 @@
       <origin xyz="0 0 0" rpy="0 1.570795 1.570795"/>
       <geometry>
-        <mesh filename="package://andbot_gazebo/robot_description/mesh/wheel-D152_SMALL.STL"/>
+        <mesh filename="package://hyperlync_robot/robot_description/mesh/wheel-D152_SMALL.STL"/>
       </geometry>
     </collision>
@@ -390,5 +390,5 @@
       <origin xyz="0 0 0" rpy="0 1.570795 1.570795"/>
       <geometry>
-        <mesh filename="package://andbot_gazebo/robot_description/mesh/wheel-D152_SMALL.STL"/>
+        <mesh filename="package://hyperlync_robot/robot_description/mesh/wheel-D152_SMALL.STL"/>
       </geometry>
        <material name="Black">
@@ -435,5 +435,5 @@
       <origin xyz="0 0 0" rpy="0 1.570795 1.570795"/>
       <geometry>
-        <mesh filename="package://andbot_gazebo/robot_description/mesh/wheel-D152_SMALL.STL"/>
+        <mesh filename="package://hyperlync_robot/robot_description/mesh/wheel-D152_SMALL.STL"/>
       </geometry>
     </collision>
@@ -441,5 +441,5 @@
       <origin xyz="0 0 0" rpy="0 1.570795 1.570795"/>
       <geometry>
-        <mesh filename="package://andbot_gazebo/robot_description/mesh/wheel-D152_SMALL.STL"/>
+        <mesh filename="package://hyperlync_robot/robot_description/mesh/wheel-D152_SMALL.STL"/>
       </geometry>
        <material name="Black">
@@ -483,5 +483,4 @@
 <!--Sonar Link -->
   <!-- Base link / sonar1 link joint -->
-<!--
   <joint name="sonar_1_fixed" type="fixed">
     <parent link="base_link"/>
@@ -489,18 +488,16 @@
     <origin xyz="0.15 0 ${0.03475+0.029}" rpy="0 0 0"/>
   </joint>
--->
 <!--Sonar Link1-->
-<!--
   <link name="sonar_1">
     <collision>
       <origin xyz="0 0 0" rpy="0 0 0"/>
       <geometry>
-        <mesh filename="package://andbot_gazebo/robot_description/mesh/sonar_HC_SR04.STL"/>
-      </geometry>
-    </collision>
-    <visual>
-      <origin xyz="0 0 0" rpy="0 0 0"/>
-      <geometry>
-        <mesh filename="package://andbot_gazebo/robot_description/mesh/sonar_HC_SR04.STL"/>
+        <mesh filename="package://hyperlync_robot/robot_description/mesh/sonar_HC_SR04.STL"/>
+      </geometry>
+    </collision>
+    <visual>
+      <origin xyz="0 0 0" rpy="0 0 0"/>
+      <geometry>
+        <mesh filename="package://hyperlync_robot/robot_description/mesh/sonar_HC_SR04.STL"/>
       </geometry>
        <material name="Yellow">
@@ -521,5 +518,4 @@
     <material>Gazebo/Yellow</material>
   </gazebo>
--->
 <!--Sonar Link 2-->
   <!-- Base link / sonar2 link joint -->
@@ -534,11 +530,11 @@
       <origin xyz="0 0 0" rpy="0 0 0"/>
       <geometry>
-        <mesh filename="package://andbot_gazebo/robot_description/mesh/sonar_HC_SR04.STL"/>
-      </geometry>
-    </collision>
-    <visual>
-      <origin xyz="0 0 0" rpy="0 0 0"/>
-      <geometry>
-        <mesh filename="package://andbot_gazebo/robot_description/mesh/sonar_HC_SR04.STL"/>
+        <mesh filename="package://hyperlync_robot/robot_description/mesh/sonar_HC_SR04.STL"/>
+      </geometry>
+    </collision>
+    <visual>
+      <origin xyz="0 0 0" rpy="0 0 0"/>
+      <geometry>
+        <mesh filename="package://hyperlync_robot/robot_description/mesh/sonar_HC_SR04.STL"/>
       </geometry>
        <material name="Yellow">
@@ -570,11 +566,11 @@
       <origin xyz="0 0 0" rpy="0 0 0"/>
       <geometry>
-        <mesh filename="package://andbot_gazebo/robot_description/mesh/sonar_HC_SR04.STL"/>
-      </geometry>
-    </collision>
-    <visual>
-      <origin xyz="0 0 0" rpy="0 0 0"/>
-      <geometry>
-        <mesh filename="package://andbot_gazebo/robot_description/mesh/sonar_HC_SR04.STL"/>
+        <mesh filename="package://hyperlync_robot/robot_description/mesh/sonar_HC_SR04.STL"/>
+      </geometry>
+    </collision>
+    <visual>
+      <origin xyz="0 0 0" rpy="0 0 0"/>
+      <geometry>
+        <mesh filename="package://hyperlync_robot/robot_description/mesh/sonar_HC_SR04.STL"/>
       </geometry>
        <material name="Yellow">
@@ -596,5 +592,4 @@
   </gazebo>
   <!-- Base link / sonar4 link joint -->
-<!--
   <joint name="sonar_4_fixed" type="fixed">
     <parent link="base_link"/>
@@ -602,18 +597,16 @@
     <origin xyz="-0.1931 0.23214 ${0.03475+0.029}"  rpy="0 0 1.5707"/>
   </joint>
--->
 <!--Sonar Link4-->
-<!--
   <link name="sonar_4">
     <collision>
       <origin xyz="0 0 0" rpy="0 0 0"/>
       <geometry>
-        <mesh filename="package://andbot_gazebo/robot_description/mesh/sonar_HC_SR04.STL"/>
-      </geometry>
-    </collision>
-    <visual>
-      <origin xyz="0 0 0" rpy="0 0 0"/>
-      <geometry>
-        <mesh filename="package://andbot_gazebo/robot_description/mesh/sonar_HC_SR04.STL"/>
+        <mesh filename="package://hyperlync_robot/robot_description/mesh/sonar_HC_SR04.STL"/>
+      </geometry>
+    </collision>
+    <visual>
+      <origin xyz="0 0 0" rpy="0 0 0"/>
+      <geometry>
+        <mesh filename="package://hyperlync_robot/robot_description/mesh/sonar_HC_SR04.STL"/>
       </geometry>
        <material name="Yellow">
@@ -634,5 +627,4 @@
     <material>Gazebo/Yellow</material>
   </gazebo>
--->
   <!-- Base link / sonar5 link joint -->
   <joint name="sonar_5_fixed" type="fixed">
@@ -646,11 +638,11 @@
       <origin xyz="0 0 0" rpy="0 0 0"/>
       <geometry>
-        <mesh filename="package://andbot_gazebo/robot_description/mesh/sonar_HC_SR04.STL"/>
-      </geometry>
-    </collision>
-    <visual>
-      <origin xyz="0 0 0" rpy="0 0 0"/>
-      <geometry>
-        <mesh filename="package://andbot_gazebo/robot_description/mesh/sonar_HC_SR04.STL"/>
+        <mesh filename="package://hyperlync_robot/robot_description/mesh/sonar_HC_SR04.STL"/>
+      </geometry>
+    </collision>
+    <visual>
+      <origin xyz="0 0 0" rpy="0 0 0"/>
+      <geometry>
+        <mesh filename="package://hyperlync_robot/robot_description/mesh/sonar_HC_SR04.STL"/>
       </geometry>
        <material name="Yellow">
@@ -682,11 +674,11 @@
       <origin xyz="0 0 0" rpy="0 0 0"/>
       <geometry>
-        <mesh filename="package://andbot_gazebo/robot_description/mesh/sonar_HC_SR04.STL"/>
-      </geometry>
-    </collision>
-    <visual>
-      <origin xyz="0 0 0" rpy="0 0 0"/>
-      <geometry>
-        <mesh filename="package://andbot_gazebo/robot_description/mesh/sonar_HC_SR04.STL"/>
+        <mesh filename="package://hyperlync_robot/robot_description/mesh/sonar_HC_SR04.STL"/>
+      </geometry>
+    </collision>
+    <visual>
+      <origin xyz="0 0 0" rpy="0 0 0"/>
+      <geometry>
+        <mesh filename="package://hyperlync_robot/robot_description/mesh/sonar_HC_SR04.STL"/>
       </geometry>
        <material name="Yellow">
@@ -708,5 +700,4 @@
   </gazebo>
   <!-- Base link / sonar7 link joint -->
-<!--
   <joint name="sonar_7_fixed" type="fixed">
     <parent link="base_link"/>
@@ -714,18 +705,16 @@
     <origin xyz="-0.37695 0 ${0.03475+0.029}"  rpy="0 0 3.14"/>
   </joint>
--->
 <!--Sonar Link7-->
-<!--
   <link name="sonar_7">
     <collision>
       <origin xyz="0 0 0" rpy="0 0 0"/>
       <geometry>
-        <mesh filename="package://andbot_gazebo/robot_description/mesh/sonar_HC_SR04.STL"/>
-      </geometry>
-    </collision>
-    <visual>
-      <origin xyz="0 0 0" rpy="0 0 0"/>
-      <geometry>
-        <mesh filename="package://andbot_gazebo/robot_description/mesh/sonar_HC_SR04.STL"/>
+        <mesh filename="package://hyperlync_robot/robot_description/mesh/sonar_HC_SR04.STL"/>
+      </geometry>
+    </collision>
+    <visual>
+      <origin xyz="0 0 0" rpy="0 0 0"/>
+      <geometry>
+        <mesh filename="package://hyperlync_robot/robot_description/mesh/sonar_HC_SR04.STL"/>
       </geometry>
        <material name="Yellow">
@@ -746,5 +735,4 @@
     <material>Gazebo/Yellow</material>
   </gazebo>
--->
   <!-- Base link / sonar8 link joint -->
   <joint name="sonar_8_fixed" type="fixed">
@@ -758,11 +746,11 @@
       <origin xyz="0 0 0" rpy="0 0 0"/>
       <geometry>
-        <mesh filename="package://andbot_gazebo/robot_description/mesh/sonar_HC_SR04.STL"/>
-      </geometry>
-    </collision>
-    <visual>
-      <origin xyz="0 0 0" rpy="0 0 0"/>
-      <geometry>
-        <mesh filename="package://andbot_gazebo/robot_description/mesh/sonar_HC_SR04.STL"/>
+        <mesh filename="package://hyperlync_robot/robot_description/mesh/sonar_HC_SR04.STL"/>
+      </geometry>
+    </collision>
+    <visual>
+      <origin xyz="0 0 0" rpy="0 0 0"/>
+      <geometry>
+        <mesh filename="package://hyperlync_robot/robot_description/mesh/sonar_HC_SR04.STL"/>
       </geometry>
        <material name="Yellow">
@@ -794,11 +782,11 @@
       <origin xyz="0 0 0" rpy="0 0 0"/>
       <geometry>
-        <mesh filename="package://andbot_gazebo/robot_description/mesh/sonar_HC_SR04.STL"/>
-      </geometry>
-    </collision>
-    <visual>
-      <origin xyz="0 0 0" rpy="0 0 0"/>
-      <geometry>
-        <mesh filename="package://andbot_gazebo/robot_description/mesh/sonar_HC_SR04.STL"/>
+        <mesh filename="package://hyperlync_robot/robot_description/mesh/sonar_HC_SR04.STL"/>
+      </geometry>
+    </collision>
+    <visual>
+      <origin xyz="0 0 0" rpy="0 0 0"/>
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