Commit message: modify urdf

File: robot_description/urdf/andbot_sonar.xacro (robot description, xacro)
@@ -21,5 +21,5 @@
       <origin xyz="0 0 -0.019" rpy="1.57 0 -1.57"/>
       <geometry>
-        <mesh filename="package://andbot_gazebo/robot_description/mesh/lidar_XV-11.STL"/>
+        <mesh filename="package://andbot/robot_description/mesh/lidar_XV-11.STL"/>
       </geometry>
     </collision>
@@ -27,5 +27,5 @@
       <origin xyz="0 0 -0.019" rpy="1.57 0 -1.57"/>
       <geometry>
-        <mesh filename="package://andbot_gazebo/robot_description/mesh/lidar_XV-11.STL"/>
+        <mesh filename="package://andbot/robot_description/mesh/lidar_XV-11.STL"/>
       </geometry>
        <material name="Green">
@@ -46,11 +46,11 @@
     <child link="xv11"/>
 <!--    plastic model     -->
-<!--	<origin xyz="-0.022 0 ${radius_wheel+0.135}" rpy="0 0 0"/>	-->
+<origin xyz="-0.022 0 ${radius_wheel+0.135}" rpy="0 0 0"/>
 <!--	metal model	-->
-<origin xyz="0.07 0 ${radius_wheel+0.135}" rpy="0 0 0"/>
+<!--	<origin xyz="0.07 0 ${radius_wheel+0.135}" rpy="0 0 0"/>-->
   </joint>
 <joint name="IMU_joint" type="fixed">
     <axis xyz="1 0 0"/>
-        <origin xyz="-0.2 0.15 0.055"/>
+        <origin xyz="0.0 0.0 0.055"/>
 	    <parent link="base_link"/>
 	    <child link="IMU_link"/>
@@ -81,5 +81,5 @@
       <origin xyz="0 0 ${radius_wheel-height_wheels_from_base}" rpy="0 0 0"/>
       <geometry>
-        <mesh filename="package://andbot_gazebo/robot_description/mesh/base_part.STL"/>
+        <mesh filename="package://andbot/robot_description/mesh/base_part.STL"/>
       </geometry>
     </collision>
@@ -87,5 +87,5 @@
       <origin xyz="0 0 ${radius_wheel-height_wheels_from_base}" rpy="0 0 0"/>
       <geometry>
-        <mesh filename="package://andbot_gazebo/robot_description/mesh/base_part.STL"/>
+        <mesh filename="package://andbot/robot_description/mesh/base_part.STL"/>
       </geometry>
        <material name="Orange">
@@ -147,11 +147,11 @@
       <origin xyz="0 0 0" rpy="0 0 0"/>
       <geometry>
-        <mesh filename="package://andbot_gazebo/robot_description/mesh/fake_body.STL"/>
-      </geometry>
-    </collision>
-    <visual>
-      <origin xyz="0 0 0" rpy="0 0 0"/>
-      <geometry>
-        <mesh filename="package://andbot_gazebo/robot_description/mesh/fake_body.STL"/>
+        <mesh filename="package://andbot/robot_description/mesh/fake_body.STL"/>
+      </geometry>
+    </collision>
+    <visual>
+      <origin xyz="0 0 0" rpy="0 0 0"/>
+      <geometry>
+        <mesh filename="package://andbot/robot_description/mesh/fake_body.STL"/>
       </geometry>
        <material name="Blue">
@@ -178,11 +178,11 @@
       <origin xyz="0 0 0" rpy="0 0 0"/>
       <geometry>
-        <mesh filename="package://andbot_gazebo/robot_description/mesh/head.STL"/>
-      </geometry>
-    </collision>
-    <visual>
-      <origin xyz="0 0 0" rpy="0 0 0"/>
-      <geometry>
-        <mesh filename="package://andbot_gazebo/robot_description/mesh/head.STL"/>
+        <mesh filename="package://andbot/robot_description/mesh/head.STL"/>
+      </geometry>
+    </collision>
+    <visual>
+      <origin xyz="0 0 0" rpy="0 0 0"/>
+      <geometry>
+        <mesh filename="package://andbot/robot_description/mesh/head.STL"/>
       </geometry>
        <material name="Blue">
@@ -224,5 +224,5 @@
       <origin xyz="0 0 0" rpy="-1.5707 1.5707 0"/>
       <geometry>
-        <mesh filename="package://andbot_gazebo/robot_description/mesh/arm_link1.STL"/>
+        <mesh filename="package://andbot/robot_description/mesh/arm_link1.STL"/>
       </geometry>
     </collision>
@@ -230,5 +230,5 @@
       <origin xyz="0 0 0" rpy="-1.5707 1.5707 0"/>
       <geometry>
-        <mesh filename="package://andbot_gazebo/robot_description/mesh/arm_link1.STL"/>
+        <mesh filename="package://andbot/robot_description/mesh/arm_link1.STL"/>
       </geometry>
        <material name="Blue">
@@ -256,5 +256,5 @@
       <origin xyz="0 0 0" rpy="-1.5707 1.5707 0"/>
       <geometry>
-        <mesh filename="package://andbot_gazebo/robot_description/mesh/arm_link2.STL"/>
+        <mesh filename="package://andbot/robot_description/mesh/arm_link2.STL"/>
       </geometry>
     </collision>
@@ -262,5 +262,5 @@
       <origin xyz="0 0 0" rpy="-1.5707 1.5707 0"/>
       <geometry>
-        <mesh filename="package://andbot_gazebo/robot_description/mesh/arm_link2.STL"/>
+        <mesh filename="package://andbot/robot_description/mesh/arm_link2.STL"/>
       </geometry>
        <material name="Blue">
@@ -288,5 +288,5 @@
       <origin xyz="0 0 0" rpy="1.57 1.5707 0"/>
       <geometry>
-        <mesh filename="package://andbot_gazebo/robot_description/mesh/arm_link1.STL"/>
+        <mesh filename="package://andbot/robot_description/mesh/arm_link1.STL"/>
       </geometry>
     </collision>
@@ -294,5 +294,5 @@
       <origin xyz="0 0 0" rpy="1.57 1.5707 0"/>
       <geometry>
-        <mesh filename="package://andbot_gazebo/robot_description/mesh/arm_link1.STL"/>
+        <mesh filename="package://andbot/robot_description/mesh/arm_link1.STL"/>
       </geometry>
        <material name="Blue">
@@ -320,5 +320,5 @@
       <origin xyz="0 0 0" rpy="-1.5707 1.5707 3.14"/>
       <geometry>
-        <mesh filename="package://andbot_gazebo/robot_description/mesh/arm_link2.STL"/>
+        <mesh filename="package://andbot/robot_description/mesh/arm_link2.STL"/>
       </geometry>
     </collision>
@@ -326,5 +326,5 @@
       <origin xyz="0 0 0" rpy="-1.5707 1.5707 0"/>
       <geometry>
-        <mesh filename="package://andbot_gazebo/robot_description/mesh/arm_link2.STL"/>
+        <mesh filename="package://andbot/robot_description/mesh/arm_link2.STL"/>
       </geometry>
        <material name="Blue">
@@ -384,5 +384,5 @@
       <origin xyz="0 0 0" rpy="0 1.570795 1.570795"/>
       <geometry>
-        <mesh filename="package://andbot_gazebo/robot_description/mesh/wheel-D152_SMALL.STL"/>
+        <mesh filename="package://andbot/robot_description/mesh/wheel-D152_SMALL.STL"/>
       </geometry>
     </collision>
@@ -390,5 +390,5 @@
       <origin xyz="0 0 0" rpy="0 1.570795 1.570795"/>
       <geometry>
-        <mesh filename="package://andbot_gazebo/robot_description/mesh/wheel-D152_SMALL.STL"/>
+        <mesh filename="package://andbot/robot_description/mesh/wheel-D152_SMALL.STL"/>
       </geometry>
        <material name="Black">
@@ -435,5 +435,5 @@
       <origin xyz="0 0 0" rpy="0 1.570795 1.570795"/>
       <geometry>
-        <mesh filename="package://andbot_gazebo/robot_description/mesh/wheel-D152_SMALL.STL"/>
+        <mesh filename="package://andbot/robot_description/mesh/wheel-D152_SMALL.STL"/>
       </geometry>
     </collision>
@@ -441,5 +441,5 @@
       <origin xyz="0 0 0" rpy="0 1.570795 1.570795"/>
       <geometry>
-        <mesh filename="package://andbot_gazebo/robot_description/mesh/wheel-D152_SMALL.STL"/>
+        <mesh filename="package://andbot/robot_description/mesh/wheel-D152_SMALL.STL"/>
       </geometry>
        <material name="Black">
@@ -483,21 +483,210 @@
 <!--Sonar Link -->
   <!-- Base link / sonar1 link joint -->
+  <joint name="sonar_6_fixed" type="fixed">
+    <parent link="base_link"/>
+    <child link="sonar_6"/>
+    <origin xyz="0.15 0 ${0.03475+0.029}" rpy="0 0 0"/>
+  </joint>
+<!--Sonar Link1-->
+  <link name="sonar_6">
+    <collision>
+      <origin xyz="0 0 0" rpy="0 0 0"/>
+      <geometry>
+        <mesh filename="package://andbot/robot_description/mesh/sonar_HC_SR04.STL"/>
+      </geometry>
+    </collision>
+    <visual>
+      <origin xyz="0 0 0" rpy="0 0 0"/>
+      <geometry>
+        <mesh filename="package://andbot/robot_description/mesh/sonar_HC_SR04.STL"/>
+      </geometry>
+       <material name="Yellow">
+         <color rgba=" 1 1 0 1"/>
+       </material>
+    </visual>
+    <inertial>
+      <origin xyz="0 0 0" rpy="0 0 0"/>
+      <mass value="0.1"/>
+      <inertia ixx="0.0135" ixy="0" ixz="0" iyy="0.0135" iyz="0" izz="0.025"/>
+    </inertial>
+  </link>
+  <gazebo reference="sonar_link6">
+    <mu1 value="2.0"/>
+    <mu2 value="2.0"/>
+    <kp value="10000000.0"/>
+    <kd value="1.0"/>
+    <material>Gazebo/Yellow</material>
+  </gazebo>
+<!--Sonar Link 2-->
+  <!-- Base link / sonar2 link joint -->
+<!--
+  <joint name="sonar_2_fixed" type="fixed">
+    <parent link="base_link"/>
+    <child link="sonar_2"/>
+    <origin xyz="0.14456 0.09192 ${0.03475+0.029}"  rpy="0 0 0"/>
+  </joint>
+-->
+<!--Sonar Link2-->
+<!--
+  <link name="sonar_2">
+    <collision>
+      <origin xyz="0 0 0" rpy="0 0 0"/>
+      <geometry>
+        <mesh filename="package://andbot/robot_description/mesh/sonar_HC_SR04.STL"/>
+      </geometry>
+    </collision>
+    <visual>
+      <origin xyz="0 0 0" rpy="0 0 0"/>
+      <geometry>
+        <mesh filename="package://andbot/robot_description/mesh/sonar_HC_SR04.STL"/>
+      </geometry>
+       <material name="Yellow">
+         <color rgba=" 1 1 0 1"/>
+       </material>
+    </visual>
+    <inertial>
+      <origin xyz="0 0 0" rpy="0 0 0"/>
+      <mass value="0.1"/>
+      <inertia ixx="0.0135" ixy="0" ixz="0" iyy="0.0135" iyz="0" izz="0.025"/>
+    </inertial>
+  </link>
+  <gazebo reference="sonar_link2">
+    <mu1 value="2.0"/>
+    <mu2 value="2.0"/>
+    <kp value="10000000.0"/>
+    <kd value="1.0"/>
+    <material>Gazebo/Yellow</material>
+  </gazebo>
+-->
+  <!-- Base link / sonar3 link joint -->
+  <joint name="sonar_7_fixed" type="fixed">
+    <parent link="base_link"/>
+    <child link="sonar_7"/>
+    <origin xyz="-0.10374 0.23695 ${0.03475+0.029}"  rpy="0 0 1.5707"/>
+  </joint>
+<!--Sonar Link3-->
+  <link name="sonar_7">
+    <collision>
+      <origin xyz="0 0 0" rpy="0 0 0"/>
+      <geometry>
+        <mesh filename="package://andbot/robot_description/mesh/sonar_HC_SR04.STL"/>
+      </geometry>
+    </collision>
+    <visual>
+      <origin xyz="0 0 0" rpy="0 0 0"/>
+      <geometry>
+        <mesh filename="package://andbot/robot_description/mesh/sonar_HC_SR04.STL"/>
+      </geometry>
+       <material name="Yellow">
+         <color rgba=" 1 1 0 1"/>
+       </material>
+    </visual>
+    <inertial>
+      <origin xyz="0 0 0" rpy="0 0 0"/>
+      <mass value="0.1"/>
+      <inertia ixx="0.0135" ixy="0" ixz="0" iyy="0.0135" iyz="0" izz="0.025"/>
+    </inertial>
+  </link>
+  <gazebo reference="sonar_link7">
+    <mu1 value="2.0"/>
+    <mu2 value="2.0"/>
+    <kp value="10000000.0"/>
+    <kd value="1.0"/>
+    <material>Gazebo/Yellow</material>
+  </gazebo>
+  <!-- Base link / sonar4 link joint -->
+<!--
+  <joint name="sonar_4_fixed" type="fixed">
+    <parent link="base_link"/>
+    <child link="sonar_4"/>
+    <origin xyz="-0.1931 0.23214 ${0.03475+0.029}"  rpy="0 0 1.5707"/>
+  </joint>
+-->
+<!--Sonar Link4-->
+<!--
+  <link name="sonar_4">
+    <collision>
+      <origin xyz="0 0 0" rpy="0 0 0"/>
+      <geometry>
+        <mesh filename="package://andbot/robot_description/mesh/sonar_HC_SR04.STL"/>
+      </geometry>
+    </collision>
+    <visual>
+      <origin xyz="0 0 0" rpy="0 0 0"/>
+      <geometry>
+        <mesh filename="package://andbot/robot_description/mesh/sonar_HC_SR04.STL"/>
+      </geometry>
+       <material name="Yellow">
+         <color rgba=" 1 1 0 1"/>
+       </material>
+    </visual>
+    <inertial>
+      <origin xyz="0 0 0" rpy="0 0 0"/>
+      <mass value="0.1"/>
+      <inertia ixx="0.0135" ixy="0" ixz="0" iyy="0.0135" iyz="0" izz="0.025"/>
+    </inertial>
+  </link>
+  <gazebo reference="sonar_link4">
+    <mu1 value="2.0"/>
+    <mu2 value="2.0"/>
+    <kp value="10000000.0"/>
+    <kd value="1.0"/>
+    <material>Gazebo/Yellow</material>
+  </gazebo>
+-->
+  <!-- Base link / sonar5 link joint -->
+  <joint name="sonar_8_fixed" type="fixed">
+    <parent link="base_link"/>
+    <child link="sonar_8"/>
+    <origin xyz="-0.27047 0.20726 ${0.03475+0.029}"  rpy="0 0 1.5707"/>
+  </joint>
+<!--Sonar Link5-->
+  <link name="sonar_8">
+    <collision>
+      <origin xyz="0 0 0" rpy="0 0 0"/>
+      <geometry>
+        <mesh filename="package://andbot/robot_description/mesh/sonar_HC_SR04.STL"/>
+      </geometry>
+    </collision>
+    <visual>
+      <origin xyz="0 0 0" rpy="0 0 0"/>
+      <geometry>
+        <mesh filename="package://andbot/robot_description/mesh/sonar_HC_SR04.STL"/>
+      </geometry>
+       <material name="Yellow">
+         <color rgba=" 1 1 0 1"/>
+       </material>
+    </visual>
+    <inertial>
+      <origin xyz="0 0 0" rpy="0 0 0"/>
+      <mass value="0.1"/>
+      <inertia ixx="0.0135" ixy="0" ixz="0" iyy="0.0135" iyz="0" izz="0.025"/>
+    </inertial>
+  </link>
+  <gazebo reference="sonar_link8">
+    <mu1 value="2.0"/>
+    <mu2 value="2.0"/>
+    <kp value="10000000.0"/>
+    <kd value="1.0"/>
+    <material>Gazebo/Yellow</material>
+  </gazebo>
+  <!-- Base link / sonar6 link joint -->
   <joint name="sonar_1_fixed" type="fixed">
     <parent link="base_link"/>
     <child link="sonar_1"/>
-    <origin xyz="-0.10374 0.23695 ${0.03475+0.029}"  rpy="0 0 1.5707"/>
-  </joint>
-<!--Sonar Link1-->
+    <origin xyz="-0.37437 0.05695 ${0.03475+0.029}"  rpy="0 0 3.14"/>
+  </joint>
+<!--Sonar Link6-->
   <link name="sonar_1">
     <collision>
       <origin xyz="0 0 0" rpy="0 0 0"/>
       <geometry>
-        <mesh filename="package://andbot_gazebo/robot_description/mesh/sonar_HC_SR04.STL"/>
-      </geometry>
-    </collision>
-    <visual>
-      <origin xyz="0 0 0" rpy="0 0 0"/>
-      <geometry>
-        <mesh filename="package://andbot_gazebo/robot_description/mesh/sonar_HC_SR04.STL"/>
+        <mesh filename="package://andbot/robot_description/mesh/sonar_HC_SR04.STL"/>
+      </geometry>
+    </collision>
+    <visual>
+      <origin xyz="0 0 0" rpy="0 0 0"/>
+      <geometry>
+        <mesh filename="package://andbot/robot_description/mesh/sonar_HC_SR04.STL"/>
       </geometry>
        <material name="Yellow">
@@ -518,23 +707,22 @@
     <material>Gazebo/Yellow</material>
   </gazebo>
-<!--Sonar Link 2-->
-  <!-- Base link / sonar2 link joint -->
+  <!-- Base link / sonar7 link joint -->
   <joint name="sonar_2_fixed" type="fixed">
     <parent link="base_link"/>
     <child link="sonar_2"/>
-    <origin xyz="-0.15374 0.23214 ${0.03475+0.029}"  rpy="0 0 1.5707"/>
-  </joint>
-<!--Sonar Link2-->
+    <origin xyz="-0.37695 0 ${0.03475+0.029}"  rpy="0 0 3.14"/>
+  </joint>
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
Commit message: add new office config

File: robot_description/urdf/andbot.xacro (robot description, xacro)
@@ -17,5 +17,5 @@
   <!-- Base footprint link-->
   <link name="base_footprint"/>
-  <link name="xv11">
+  <link name="rplidar">
     <collision>
       <origin xyz="0 0 -0.019" rpy="1.57 0 -1.57"/>
@@ -39,10 +39,10 @@
     </inertial>
   </link>
-  <gazebo reference="xv11">
+  <gazebo reference="rplidar">
     <material>Gazebo/Green</material>
   </gazebo>
-  <joint name="xv11_fixed" type="fixed">
+  <joint name="rplidar_fixed" type="fixed">
     <parent link="base_footprint"/>
-    <child link="xv11"/>
+    <child link="rplidar"/>
 <!--    plastic model     -->
 <origin xyz="-0.022 0 ${radius_wheel+0.135}" rpy="0 0 0"/>
@@ -979,9 +979,9 @@
   </gazebo>
 <!-- xv11 plugin -->
-  <gazebo reference="xv11">
+  <gazebo reference="rplidar">
     <mu1>1.0</mu1>
     <mu2>1.0</mu2>
     <material>Gazebo/Blue</material>
-    <sensor type="ray" name="xv11_sensor">
+    <sensor type="ray" name="rplidar_sensor">
       <pose>0 0 0 0 0 0</pose>
       <visualize>true</visualize>
@@ -1014,6 +1014,6 @@
       </ray>
       <plugin name="gazebo_ros_head_hokuyo_controller" filename="libgazebo_ros_laser.so">
-        <topicName>xv11_scan</topicName>
-        <frameName>xv11</frameName>
+        <topicName>rplidar_scan</topicName>
+        <frameName>rplidar</frameName>
       </plugin>
     </sensor>
